File: el84_tran1/el84_tran1.kicad_sch (KiCad schematic)
At the start: 9 parts, among them T2 PYE_PJ105, U1 EL41

Commit message: redone the el41 spice model, added library directory
Parts:
- R2: value 188 -> 1600
- R4: value 240 -> 220
- U1: value EL41 -> el41
- Vdd1: value 230 -> 250
Other:
- note removed: "peak to peak load current for R2 change 1600R 234mAs 188R 251mAs"
Changed lines of the file:
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@@
-		)
-	)
-	(text "peak to peak load current for R2 change\n1600R 234mAs\n188R  251mAs"
-		(exclude_from_sim yes)
-		(at 195.58 83.312 0)
-		(effects
-			(font
-				(size 1.27 1.27)
-			)
 		)
 	)
@@
 				)
 			)
+			(project "el84_tran1"
+				(path "/b4564891-33ed-48ee-b520-9a9da1c282d1"
+					(reference "#GND05")
+					(unit 1)
+				)
+			)
 		)
 	)
@@
 			)
 		)
-		(property "Value" "240"
+		(property "Value" "220"
 			(at 121.92 139.6999 0)
 			(effects
@@
 				)
 			)
+			(project "el84_tran1"
+				(path "/b4564891-33ed-48ee-b520-9a9da1c282d1"
+					(reference "Rk1")
+					(unit 1)
+				)
+			)
 		)
 	)
@@
 				)
 			)
+			(project "el84_tran1"
+				(path "/b4564891-33ed-48ee-b520-9a9da1c282d1"
+					(reference "#GND06")
+					(unit 1)
+				)
+			)
 		)
 	)
@@
 				)
 			)
+			(project "el84_tran1"
+				(path "/b4564891-33ed-48ee-b520-9a9da1c282d1"
+					(reference "C1")
+					(unit 1)
+				)
+			)
 		)
 	)
@@
 				)
 			)
+			(project "el84_tran1"
+				(path "/b4564891-33ed-48ee-b520-9a9da1c282d1"
+					(reference "#GND01")
+					(unit 1)
+				)
+			)
 		)
 	)
@@
 			)
 		)
-		(property "Value" "188"
+		(property "Value" "1600"
 			(at 172.72 92.7099 0)
 			(effects
@@
 				)
 			)
+			(project "el84_tran1"
+				(path "/b4564891-33ed-48ee-b520-9a9da1c282d1"
+					(reference "Rs1")
+					(unit 1)
+				)
+			)
 		)
 	)
@@
 				)
 			)
+			(project "el84_tran1"
+				(path "/b4564891-33ed-48ee-b520-9a9da1c282d1"
+					(reference "V1")
+					(unit 1)
+				)
+			)
 		)
 	)
@@
 			(project "el41_trans1"
 				(path "/842534cd-cf97-4a2e-b074-ba30f85f02b8"
+					(reference "#GND04")
+					(unit 1)
+				)
+			)
+			(project "el84_tran1"
+				(path "/b4564891-33ed-48ee-b520-9a9da1c282d1"
 					(reference "#GND04")
 					(unit 1)
@@
 				)
 			)
+			(project "el84_tran1"
+				(path "/b4564891-33ed-48ee-b520-9a9da1c282d1"
+					(reference "T2")
+					(unit 1)
+				)
+			)
 		)
 	)
@@
 			)
 		)
-		(property "Value" "EL41"
+		(property "Value" "el41"
 			(at 127 100.076 0)
 			(effects
@@
 			)
 		)
-		(property "Datasheet" "http://www.r-type.org/pdfs/el84.pdf"
+		(property "Datasheet" ""
 			(at 121.92 109.22 0)
 			(effects
@@
 			)
 		)
-		(property "Description" "pentode, 12W"
+		(property "Description" "pentode, 9W"
 			(at 121.92 109.22 0)
 			(effects
@@
 			)
 		)
-		(property "Sim.Name" "EL41_2"
+		(property "Sim.Name" "EL41"
 			(at 121.92 109.22 0)
 			(effects
@@
 				)
 			)
+			(project "el84_tran1"
+				(path "/b4564891-33ed-48ee-b520-9a9da1c282d1"
+					(reference "U1")
+					(unit 1)
+				)
+			)
 		)
 	)
@@
 				)
 			)
+			(project "el84_tran1"
+				(path "/b4564891-33ed-48ee-b520-9a9da1c282d1"
+					(reference "#GND02")
+					(unit 1)
+				)
+			)
 		)
 	)
@@
 				)
 			)
+			(project "el84_tran1"
+				(path "/b4564891-33ed-48ee-b520-9a9da1c282d1"
+					(reference "Rl1")
+					(unit 1)
+				)
+			)
 		)
 	)
@@
 			)
 		)
-		(property "Value" "230"
+		(property "Value" "250"
 			(at 209.55 124.3301 0)
 			(effects
@@
 				)
 			)
+			(project "el84_tran1"
+				(path "/b4564891-33ed-48ee-b520-9a9da1c282d1"
+					(reference "Vdd1")
+					(unit 1)
+				)
+			)
 		)
 	)
@@
 					(reference "R1")
 					(unit 1)
+				)
+			)
+			(project "el84_tran1"
+				(path "/b4564891-33ed-48ee-b520-9a9da1c282d1"
+					(reference "R1")
+					(unit 1)
